Commit message: working on figuring out what is wrong with the real hand. simulation is working just fine with my IK class

File: pc_testing_code/sim/hand_arm.urdf (robot description, URDF)
Before this commit: robot udp_hand_arm, 8 links, 7 joints
Links:
- link finger1_link: geometry collision box size=0.015 0.015 0.07; visual box size=0.015 0.015 0.07
- link finger2_link: geometry collision box size=0.015 0.015 0.07; visual box size=0.015 0.015 0.07
- link palm_link: geometry collision box size=0.06 0.04 0.03; visual box size=0.06 0.04 0.03
Joints:
- joint elbow_angle: limit lower=-1.57079632679 upper=1.57079632679 effort=40 velocity=3.0 -> lower=-5 upper=5 effort=40 velocity=3.0; origin xyz=0.30 0 0 rpy=0 0 0 -> xyz=0 0 0.30 rpy=0 0 0
- joint finger1: axis 0 0 1 -> 1 0 0; origin xyz=0.03 0.02 0 rpy=0 0 0 -> xyz=0 0.01 0.03 rpy=0 0 0
- joint finger2: axis 0 0 1 -> 1 0 0; origin xyz=0.03 -0.02 0 rpy=0 0 0 -> xyz=0 -0.01 0.03 rpy=0 0 0
- joint wrist_angle: origin xyz=0.20 0 0 rpy=0 0 0 -> xyz=0 0 0.20 rpy=0 0 0
- joint wrist_rotation: axis 1 0 0 -> 0 0 1; origin xyz=0.05 0 0 rpy=0 0 0 -> xyz=0 0 0.05 rpy=0 0 0
